File: ZX Interface 1 ROM 39SF010.kicad_sch (KiCad schematic)
At the start: 14 parts, among them J2 Conn_01x09_Pin, J3 BBL-112-G-E, J4 BBL-112-G-E, SW1 SW_SPDT, U1 SST39SF040A TSOP

Commit message: Add files via upload
Parts:
- renumbered J2 to J1
Changed lines of the file:
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@@
     (rev "1.1")
     (company "Andy Potter")
-    (comment 1 "Add 0V connection to J2 allowing external switching of A14/A15/A16/A17 and A18.")
+    (comment 1 "Add 0V connection to J1 allowing external switching of A14/A15/A16/A17 and A18.")
     (comment 2 "DO NOT EXTERNALLY SWITCH A13")
   )
@@
   (symbol (lib_id "Connector:Conn_01x09_Pin") (at 205.994 16.764 90) (mirror x) (unit 1)
     (in_bom yes) (on_board yes) (dnp no)
-    (property "Reference" "J2" (at 217.17 18.034 90)
+    (property "Reference" "J1" (at 217.17 18.034 90)
       (effects (font (size 1.27 1.27)))
     )
@@
       (project "ZX Interface 1 ROM 39SF010"
         (path "/8751c651-26dc-4d30-8f2d-d9f24098bdc5"
-          (reference "J2") (unit 1)
-        )
-      )
+          (reference "J1") (unit 1)
+        )
+      )

Commit message: Updated to use Right Angle 9 pin Header
Parts:
- J1: footprint Connector_PinSocket_2.54mm:PinSocket_1x09_P2.54mm_Vertical -> Switch:PinSocket_1x09_P2.54mm_HorizontalR
Changed lines of the file:
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@@
       (effects (font (size 1.27 1.27)) hide)
     )
-    (property "Footprint" "Connector_PinSocket_2.54mm:PinSocket_1x09_P2.54mm_Vertical" (at 205.994 16.764 0)
+    (property "Footprint" "Switch:PinSocket_1x09_P2.54mm_HorizontalR" (at 205.994 16.764 0)
       (effects (font (size 1.27 1.27)) hide)
     )

Commit message: Add files via upload
Updated file to Kicad 9. Restructured folders. Added ibom (Interactive BOM)
Parts:
- C1: footprint Capacitor_SMD:C_1206_3216Metric_Pad1.33x1.80mm_HandSolder -> Mod:C_1206_3216Metric_Pad1.33x1.80mm_HandSolder; symbol Device:C -> IF1_Replacement_ROM:C
- J1: footprint Switch:PinSocket_1x09_P2.54mm_HorizontalR -> Mod:PinSocket_1x09_P2.54mm_HorizontalR; symbol Connector:Conn_01x09_Pin -> IF1_Replacement_ROM:Conn_01x09_Pin
- J3, J4: footprint Switch:Pin-Pin Header 2.54mm Round Samtec BBL-112-G-E -> Mod:Pin-Pin Header 2.54mm Round Samtec BBL-112-G-E; symbol PinPIn12:BBL-112-G-E -> IF1_Replacement_ROM:BBL-112-G-E
- R1, R2, R3, R4, R5, R6, R7, R8: footprint Resistor_SMD:R_1206_3216Metric_Pad1.30x1.75mm_HandSolder -> Mod:R_1206_3216Metric_Pad1.30x1.75mm_HandSolder; symbol Device:R -> IF1_Replacement_ROM:R
- SW1: footprint Switch:SW_PCM12SMTR -> Mod:SW_PCM12SMTR; symbol Switch:PCM12SMTR -> IF1_Replacement_ROM:PCM12SMTR
- U1: footprint Package_SO:TSOP-I-32_12.4x8mm_P0.5mm -> Mod:TSOP-I-32_12.4x8mm_P0.5mm; symbol Memory_Flash:SST39SF010 -> IF1_Replacement_ROM:SST39SF010
Other:
- note added: "J1 pin 1 ~WE pulled high in operation by 10K resistor R1 on ROM board. J1 pin 2 A18 pulled high in operation by 10K resistor R8 on ROM board. J1 pin 3 A17 pulled high in operation by 10K resistor R7 on ROM board. J1 pin 4 A16 selects ROM to use, pulled high or low in operation by switch and 10K resistor R2 on ROM board. Includes switching of A16 if internal switch set to position B. J1 pin 5 A15 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"
- note removed: "J1 pin 1 ~WE pulled high in operation by 10K resistor R1 on ROM board. J1 pin 2 A18 pulled high in operation by 10K resistor R8 on ROM board. J1 pin 3 A17 pulled high in operation by 10K resistor R7 on ROM board. J1 pin 4 A16 selects ROM to use, pulled high or low in operation by switch and 10K resistor R2 on ROM board. J1 pin 5 A15 pulled high in operation by 10K resistor R5 on ROM board. J1 pin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"
